File: PartoDos/PartoDos.kicad_pcb (KiCad board)
At the start: 2 copper layers, 80 x 100.2 mm, 58 parts, among them J1 RED4, J10 WHI4, J11 RED5, J12 GRE3, J13 GNC_BOND, J14 GNC_BOND, J15 GNC_BOND, J16 GNC_BOND, J17 GNC_BOND, J18 GNC_BOND, J19 GNC_BOND, J2 YEL4, J20 GNC_BOND, J21 GNC_BOND, J22 GNC_BOND, J23 GNC_BOND, J24 GNC_BOND, J25 GNC_BOND, J26 GNC_BOND, J27 GNC_BOND, J28 GNC_BOND, J29 GNC_BOND, J3 BLU1, J30 GNC_BOND, J31 GNC_BOND, J32 GNC_BOND, J33 GNC_BOND, J34 GNC_BOND, J4 YEL3, J5 GRE1, J6 WHI3, J7 GRE2, J8 BLU2, J9 YEL5

Commit message: Fixed code
Had an issue in shiftOutData where I defined the wrong data type (16 bit instead of 32 bit) so it cut all data short
Parts:
- removed J20, J22: GNC_BOND, Connector_Wire:SolderWirePad_1x01_SMD_1x2mm
- added D13: WHI, LED_SMD:LED_0805_2012Metric, B.Cu at (140.5, 55.5)
- added D14: WHI, LED_SMD:LED_0805_2012Metric, F.Cu at (140.5, 55.5)
- added R13: 1, Resistor_SMD:R_1206_3216Metric, B.Cu at (137.2, 58.4)
- added R14: 1, Resistor_SMD:R_1206_3216Metric, F.Cu at (137.2, 58.4)
- J15: moved to B.Cu
- J27: value GNC_BOND -> TOP_STAR_VCC
- moved J15 11.4 mm to (138.9, 76.3), turned to 180 degrees
Connections:
- J27 pad 1: GND -> Net-(J27-Pad1)
Routing:
- net Net-(J27-Pad1): track 0.00 -> 31.8 mm, vias 0 -> 1
- net GND: track 28.7 -> 31.6 mm
- net Net-(D14-Pad2): track 0.00 -> 2.64 mm
- net Net-(D13-Pad2): track 0.00 -> 2.64 mm
- net /WHI4: track 22.4 -> 21.9 mm
